File: RP-Link.kicad_sch (KiCad schematic)
At the start: 31 parts, among them J1 TYPE-C_16P, J2 Conn_01x06, SW1 SKRKAEE020_SMD, U1 W25Q16JVUX, U2 ME6211C33M5G, U3 RP2040, Y1 Crystal_GND24

Commit message: 修复一些问题
#2
Parts:
- added D2: D_Schottky, Diode_SMD:D_SOD-123F, symbol Device:D_Schottky
- C1, C10, C11, C12, C13, C14, C15, C2, C5, C6, C7, C8, C9: footprint Capacitor_SMD:C_0603_1608Metric -> Capacitor_SMD:C_0402_1005Metric
- C3, C4: footprint Capacitor_SMD:C_0402_1005Metric -> Capacitor_SMD:C_0603_1608Metric
- R1, R4, R5, R6, R7, R8: footprint Resistor_SMD:R_0603_1608Metric -> Resistor_SMD:R_0402_1005Metric
Connections:
- net +3.3V: no longer J2.1 (Pin_1)
- net GPIO2: now also J2.6 (Pin_6); no longer J2.3 (Pin_3)
- net GPIO3: now also J2.5 (Pin_5); no longer J2.4 (Pin_4)
- net GPIO4: now also J2.4 (Pin_4); no longer J2.5 (Pin_5)
- net GPIO5: now also J2.3 (Pin_3); no longer J2.6 (Pin_6)
- net VBUS: now also D2.2 (A); no longer C3.1, U2.1 (VIN), U2.3 (EN)
- new net VCC: C3.1, D2.1 (K), J2.1 (Pin_1), U2.1 (VIN), U2.3 (EN)
